File: capacity_measurement.kicad_pcb (KiCad board)
At the start: 2 copper layers, 68 parts, among them J1 Conn_01x02, SW1 SW_Push, U1 nRF52832-QFxx, U2 AMS1117-3.3, U3 SX1308, U4 TP4056, U5 MC34063AD, U6 HT7127-1-SOT89, U7 TagConnect, U8 WX-DC12003, Y1 32MHz

Commit message: wip
Parts:
- added J2: Ultrasound, Connector_PinHeader_2.54mm:PinHeader_1x04_P2.54mm_Vertical, F.Cu at (116.7, 84.9)
- added U9: Temp, Package_TO_SOT_THT:TO-92_Inline, F.Cu at (121.0, 85.8)

Commit message: wip
Parts:
- removed TH1: NTC, smdpad:smdpad_01x02_1.27_2.54_0.51
- added C19: 10uF, Capacitor_SMD:C_0805_2012Metric, F.Cu at (240.2, 77.2)
- added C21: >=23uF, Capacitor_THT:CP_Radial_D10.0mm_P5.00mm, F.Cu at (201.0, 142.5)
- added C22: 10uF, Capacitor_SMD:C_0201_0603Metric, F.Cu at (219.5, 138.7)
- added C23: 1uF, Capacitor_SMD:C_0201_0603Metric, F.Cu at (235.2, 92.7)
- added C24: 1uF, Capacitor_SMD:C_0201_0603Metric, F.Cu at (249.0, 71.2)
- added C25: 1uF, Capacitor_SMD:C_0201_0603Metric, F.Cu at (249.0, 69.5)
- added C26: C, Capacitor_SMD:C_0201_0603Metric, F.Cu at (233.6, 106.9)
- added C27: C, Capacitor_SMD:C_0201_0603Metric, F.Cu at (236.1, 106.9)
- added Csd1: CP, Capacitor_SMD:C_Elec_6.3x5.4, F.Cu at (45.5, 63.2)
- added D3: LED_BARG, LED_SMD:LED_RGB_1210, F.Cu at (232.9, 84.4)
- added D5: LED, LED_SMD:LED_1210_3225Metric, F.Cu at (185.4, 83.2)
- added D6: LED, LED_SMD:LED_1210_3225Metric, F.Cu at (41.9, 34.5)
- added D7: LED, LED_SMD:LED_1210_3225Metric, F.Cu at (41.9, 37.8)
- added J10: Conn_01x10, Connector_PinHeader_2.54mm:PinHeader_1x10_P2.54mm_Vertical, F.Cu at (41.4, 26.9)
- added J11: Conn_01x08, Connector_PinHeader_2.54mm:PinHeader_1x08_P2.54mm_Vertical, F.Cu at (68.3, 26.9)
- added J12: Conn_01x03, smdpad:smdpad_01x03_1.27_2.54_0.51, F.Cu at (273.1, 124.0)
- added J13: Conn_01x03, smdpad:smdpad_01x03_1.27_2.54_0.51, F.Cu at (279.9, 121.3)
- added J14: Conn_01x03, smdpad:smdpad_01x03_1.27_2.54_0.51, F.Cu at (272.3, 127.5)
- added J3: PWR_CONN, smdpad:smdpad_02x05_1.27_2.54_0.51, F.Cu at (263.7, 119.6)
- added J4: USB_B_Micro, Connector_USB:USB_Micro-B_Molex_47346-0001, F.Cu at (25.7, 35.6)
- added J5: Micro_SD_Card, aliexpress:microSD, F.Cu at (31.2, 63.8)
- added J6: Conn_01x08, smdpad:smdpad_01x08_1.27_2.54_0.51, F.Cu at (259.0, 136.2)
- added J7: Conn_01x12, smdpad:smdpad_01x12_1.27_2.54_0.51, F.Cu at (244.8, 49.9)
- added J8: Conn_01x08, Connector_PinHeader_2.54mm:PinHeader_1x08_P2.54mm_Vertical, F.Cu at (50.5, 75.2)
- added J9: Conn_01x06, Connector_PinHeader_2.54mm:PinHeader_1x06_P2.54mm_Vertical, F.Cu at (73.4, 75.2)
- added JP10: Temp_NTC, Jumper:SolderJumper-3_P1.3mm_Bridged12_RoundedPad1.0x1.5mm, F.Cu at (279.8, 127.5)
- added JP11: Bridge3, Jumper:SolderJumper-3_P1.3mm_Bridged12_RoundedPad1.0x1.5mm, F.Cu at (173.6, 91.1)
- added JP5: AOP_EN, Jumper:SolderJumper-2_P1.3mm_Open_TrianglePad1.0x1.5mm, F.Cu at (272.3, 57.8)
- added JP6: TempEN, Jumper:SolderJumper-2_P1.3mm_Bridged_RoundedPad1.0x1.5mm, F.Cu at (249.0, 77.5)
- added JP7: shunt, Jumper:SolderJumper-2_P1.3mm_Open_TrianglePad1.0x1.5mm, F.Cu at (215.1, 133.6)
- added JP8: Vbat, Jumper:SolderJumper-3_P1.3mm_Bridged12_RoundedPad1.0x1.5mm, B.Cu at (214.6, 134.6)
- added JP9: Bridge2, Jumper:SolderJumper-3_P1.3mm_Bridged12_RoundedPad1.0x1.5mm, F.Cu at (179.3, 88.6)
- added Q1: 2N7002, Package_TO_SOT_SMD:SOT-23, F.Cu at (44.5, 57.7)
- added Q2: 2N7002, Package_TO_SOT_SMD:SOT-23, F.Cu at (254.1, 54.0)
- added Q3: 2N7002, Package_TO_SOT_SMD:SOT-23, F.Cu at (245.8, 60.8)
- added R13: R, Resistor_SMD:R_0805_2012Metric, F.Cu at (263.5, 60.5)
- added R14: R, Resistor_SMD:R_0805_2012Metric, F.Cu at (263.5, 63.4)
- added R15: R, Resistor_SMD:R_0805_2012Metric, F.Cu at (267.9, 54.6)
- added R16: R, Resistor_SMD:R_0805_2012Metric, F.Cu at (254.7, 63.6)
- added R17: R, Resistor_SMD:R_0805_2012Metric, F.Cu at (250.3, 63.6)
- added R18: R, Resistor_SMD:R_0805_2012Metric, F.Cu at (254.7, 60.7)
- added R19: R, Resistor_SMD:R_0805_2012Metric, F.Cu at (259.1, 60.5)
- added R20: R, Resistor_SMD:R_0805_2012Metric, F.Cu at (263.5, 57.5)
- added R21: R, Resistor_SMD:R_0805_2012Metric, F.Cu at (263.5, 54.6)
- added R22: R, Resistor_SMD:R_0805_2012Metric, F.Cu at (259.1, 57.5)
- added R23: 75K 1%, Resistor_SMD:R_0805_2012Metric, F.Cu at (250.3, 60.0)
- added R24: R, Resistor_SMD:R_0805_2012Metric, F.Cu at (258.5, 54.6)
- added R25: R, Resistor_SMD:R_0805_2012Metric, F.Cu at (254.7, 57.7)
- added R26: 10k, Resistor_SMD:R_0805_2012Metric, F.Cu at (202.8, 95.8)
- added R27: 37k, Resistor_SMD:R_0805_2012Metric, F.Cu at (196.3, 112.0)
- added R28: 5k, Resistor_SMD:R_0805_2012Metric, F.Cu at (192.8, 112.0)
- added R29: R, Resistor_SMD:R_0805_2012Metric, F.Cu at (238.5, 86.7)
- added R30: R, Resistor_SMD:R_0805_2012Metric, F.Cu at (244.6, 80.2)
- added R31: 10k, Resistor_SMD:R_0805_2012Metric, F.Cu at (242.9, 83.2)
- added R32: 0.4, Resistor_SMD:R_0805_2012Metric, F.Cu at (238.5, 83.7)
- added R33: 1k, Resistor_SMD:R_0805_2012Metric, F.Cu at (240.2, 80.2)
- added R34: 1k, Resistor_SMD:R_0805_2012Metric, F.Cu at (244.7, 77.2)
- added R35: 0.45, Resistor_SMD:R_0805_2012Metric, F.Cu at (212.6, 133.6)
- added R36: 1k, Resistor_SMD:R_0805_2012Metric, F.Cu at (212.6, 136.7)
- added R37: 3.4k, Resistor_SMD:R_0805_2012Metric, F.Cu at (209.0, 137.7)
- added R38: R, Resistor_SMD:R_0805_2012Metric, F.Cu at (234.6, 104.6)
- added R39: R, Resistor_SMD:R_0805_2012Metric, F.Cu at (173.0, 94.6)
- added R40: R, Resistor_SMD:R_0805_2012Metric, F.Cu at (184.7, 86.8)
- added R41: R, Resistor_SMD:R_0805_2012Metric, F.Cu at (37.6, 35.3)
- added R42: R, Resistor_SMD:R_0805_2012Metric, F.Cu at (37.6, 37.3)
- added TH2: NTC, smdpad:smdpad_01x02_1.27_2.54_0.51, F.Cu at (241.8, 86.4)
- added U10: TP4056, Package_SO:SOP-8_3.76x4.96mm_P1.27mm, F.Cu at (233.7, 79.0)
- added U11: MC34063AD, Package_SO:SOIC-8_3.9x4.9mm_P1.27mm, F.Cu at (206.8, 133.7)
- added U12: HT7127-1-SOT89, Package_TO_SOT_SMD:SOT-89-3_Handsoldering, F.Cu at (223.0, 141.7)
- added U13: AMS1117-2.85, Package_TO_SOT_SMD:SOT-223-3_TabPin2, F.Cu at (220.7, 133.6)
- added U14: ADXL343, Package_LGA:LGA-14_3x5mm_P0.8mm_LayoutBorder1x6y, F.Cu at (231.7, 95.1)
- added U15: BMP280, Package_LGA:Bosch_LGA-8_2x2.5mm_P0.65mm_ClockwisePinNumbering, F.Cu at (245.7, 70.4)
- added U16: CP2102N-A01-GQFN24, Package_DFN_QFN:QFN-24-1EP_4x4mm_P0.5mm_EP2.6x2.6mm, F.Cu at (237.6, 118.4)
- added Y2: 32MHz, Crystal:Crystal_HC18-U_Vertical, F.Cu at (78.5, 38.1)
- BT1: value bat -> Bat; footprint Connector_PinSocket_2.54mm:PinSocket_1x02_P2.54mm_Vertical -> Connector_PinHeader_2.54mm:PinHeader_1x02_P2.54mm_Vertical
- C1, C2: value 12pF -> 0.1uF
- C10: value 100nF -> 100pF
- C11: value 100nF -> NC
- C12: value 22uF -> 100nF
- C13: value >=23uF -> 0.8pF; footprint Capacitor_SMD:C_0805_2012Metric -> Capacitor_SMD:C_0201_0603Metric
- C14, C15: value 22uF -> 12pF
- C16: value 10uF -> NC; footprint Capacitor_SMD:C_0805_2012Metric -> Capacitor_SMD:C_0201_0603Metric
- C17: value 280pF -> 22uF
- C18: value 10uF -> 22uF
- C20: value NC -> 280pF
- C3: value 0.8pF -> C
- C4: value 100nF -> C
- C5: value NC -> 100nF
- C6: value 100pF -> 100nF
- C7: value 1uF -> 4.7uF; footprint Capacitor_SMD:C_0201_0603Metric -> Capacitor_SMD:C_0805_2012Metric
- C9: value 4.7uF -> 1uF; footprint Capacitor_SMD:C_0805_2012Metric -> Capacitor_SMD:C_0201_0603Metric
- H1, H2, H3, H4: footprint MountingHole:MountingHole_2.2mm_M2_Pad -> MountingHole:MountingHole_2.2mm_M2_DIN965_Pad
- J1: value Conn_01x02 -> Ultrasound; footprint smdpad:smdpad_01x02_2.54_3.81_2.54 -> Connector_PinHeader_2.54mm:PinHeader_1x04_P2.54mm_Vertical
- J2: value Ultrasound -> Conn_01x02; footprint Connector_PinHeader_2.54mm:PinHeader_1x04_P2.54mm_Vertical -> smdpad:smdpad_01x02_2.54_3.81_2.54
- JP1: value Boost -> USB_5V; footprint Jumper:SolderJumper-3_P1.3mm_Bridged12_RoundedPad1.0x1.5mm -> Jumper:SolderJumper-2_P1.3mm_Bridged_RoundedPad1.0x1.5mm
- JP2: value TempEN -> Bridge1; footprint Jumper:SolderJumper-2_P1.3mm_Bridged_RoundedPad1.0x1.5mm -> Jumper:SolderJumper-3_P1.3mm_Bridged12_RoundedPad1.0x1.5mm; moved to F.Cu
- JP3: value shunt -> SD_EN; moved to B.Cu
- JP4: value Reg_select -> AOP_EN; footprint Jumper:SolderJumper-3_P1.3mm_Bridged12_RoundedPad1.0x1.5mm -> Jumper:SolderJumper-2_P1.3mm_Open_TrianglePad1.0x1.5mm; moved to F.Cu
- L1: value 3.9nH -> 10uH; moved to B.Cu
- L3: value 10uH -> 3.9nH; moved to F.Cu
- R1, R6: value 10k -> R
- R10: value 0.45 -> R
- R11, R8, R9: value 1k -> R
- R12: value 3.4k -> R
- R2: value 37k -> R
- R3: value 5k -> R
- R4, R5: moved to F.Cu
- R7: value 0.4 -> R
- SC1: footprint Connector_PinSocket_2.54mm:PinSocket_1x02_P2.54mm_Vertical -> smdpad:smdpad_01x02_1.27_2.54_0.51
- TP1: value Reset -> Vmcu
- TP2: value XC1 -> XC2; moved to F.Cu
- TP3: value XC2 -> XC1; moved to F.Cu
- TP4: value Vnrf -> Reset; moved to F.Cu
- U1: value nRF52832-QFxx -> WX-DC12003; footprint Package_DFN_QFN:QFN-48-1EP_6x6mm_P0.4mm_EP4.6x4.6mm -> aliexpress:WX-DC12003_vertical
- U2: value AMS1117-3.3 -> AMS1117-5.0; moved to B.Cu
- U3: value SX1308 -> DS18B20; footprint aliexpress:SX1308 -> Package_TO_SOT_THT:TO-92_Inline
- U4: value TP4056 -> ULN2003; footprint Package_SO:SOP-8_3.76x4.96mm_P1.27mm -> Package_SO:STC_SOP-16_3.9x9.9mm_P1.27mm
- U5: value MC34063AD -> Opamp_Dual_Generic; footprint Package_SO:SOIC-8_3.9x4.9mm_P1.27mm -> Package_SO:SSOP-8_3.95x5.21x3.27mm_P1.27mm
- U6: value HT7127-1-SOT89 -> MPR121; footprint Package_TO_SOT_SMD:SOT-89-3_Handsoldering -> Package_DFN_QFN:Texas_S-PWQFN-N20
- U7: value TagConnect -> nRF52832-QFxx; footprint Connector:Tag-Connect_TC2030-IDC-NL_2x03_P1.27mm_Vertical -> Package_DFN_QFN:QFN-48-1EP_6x6mm_P0.4mm_EP4.6x4.6mm; moved to F.Cu
- U8: value WX-DC12003 -> TagConnect; footprint aliexpress:WX-DC12003_vertical -> Connector:Tag-Connect_TC2030-IDC-NL_2x03_P1.27mm_Vertical
- U9: value Temp -> SX1308; footprint Package_TO_SOT_THT:TO-92_Inline -> aliexpress:SX1308
- Y1: value 32MHz -> 32.768k; footprint Crystal:Crystal_HC18-U_Vertical -> Crystal:Crystal_C38-LF_D3.0mm_L8.0mm_Vertical
- moved C2 160.4 mm to (271.6, 49.0), turned to 0 degrees
- moved R7 154.3 mm to (284.8, 129.1), turned to 0 degrees
- moved J2 153.5 mm to (264.3, 126.9)
- moved U4 151.2 mm to (276.8, 140.1)
- moved JP1 139.1 mm to (30.7, 34.3), turned to 180 degrees
- moved D1 134.1 mm to (275.4, 120.0)
- moved C1 132.5 mm to (244.8, 63.9), turned to 0 degrees
- moved JP3 128.1 mm to (42.9, 61.0), turned to 0 degrees
- moved R9 120.2 mm to (47.2, 57.7), turned to 90 degrees
- moved C20 114.3 mm to (206.3, 136.9), turned to 180 degrees
- moved U8 112.9 mm to (79.0, 59.9), turned to 180 degrees
- moved U2 111.2 mm to (203.7, 132.8)
- moved JP4 111.1 mm to (267.9, 60.8), turned to 0 degrees
- moved R10 108.5 mm to (272.3, 54.6), turned to 0 degrees
- moved TP3 106.7 mm to (214.5, 94.0)
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Connections:
- AE1 pad 1: /ANT -> /mcu/ANT
- C10 pad 1: /Vnrf -> GND
- C10 pad 2: GND -> /mcu/DEC3
- C11 pad 1: /Vnrf -> GND
- C11 pad 2: GND -> /mcu/DEC2
- C12 pad 1: /Vboost_in -> GND
- C12 pad 2: GND -> /mcu/DEC1
- C13 pad 1: GNDD -> /mcu/RF_out
- C14 pad 1: +3V3 -> Net-(C14-Pad1)
- C15 pad 1: +5V -> Net-(C15-Pad1)
- C16 pad 1: /Vbat -> /mcu/ANT
- C17 pad 1: /BB_TC -> +5V
- C17 pad 2: GNDD -> GND
- C18 pad 1: +2V8 -> +12V
- C2 pad 1: Net-(C2-Pad1) -> +2V8
- C20 pad 1: /ANT -> /solar/BB_TC
- C20 pad 2: GND -> +5V
- C3 pad 1: /RF_out -> /P00
- C4 pad 1: GND -> /P01
- C4 pad 2: /DEC1 -> GND
- C5 pad 1: GND -> +2V8
- C5 pad 2: /DEC2 -> GND
- C6 pad 1: GND -> +2V8
- C6 pad 2: /DEC3 -> GND
- C7 pad 1: GND -> +2V8
- C7 pad 2: /DEC4 -> GND
- C8 pad 1: /Vnrf -> +2V8
- C9 pad 1: /Vnrf -> GND
- C9 pad 2: GND -> /mcu/DEC4
- D1 pad 2: /TP4056_Vcc -> +2V8
- D2 pad 1: +5V -> +12V
- D2 pad 2: /Boost_SW -> /dc_boost/Boost_SW
- D4 pad 1: /BB_SWE -> /solar/BB_SWE
- J1 pad 1: Net-(J1-Pad1) -> GND
- J1 pad 2: Net-(J1-Pad2) -> /US_ECHO
- J2 pad 1: GND -> Net-(J2-Pad1)
- J2 pad 2: /US_ECHO -> Net-(J2-Pad2)
- JP1 pad 1: +3V3 -> +5V
- JP1 pad 2: /Vboost_in -> /ftdi/Vusb
- JP2 pad 1: GND -> +5V
- JP2 pad 2: Net-(JP2-Pad2) -> Net-(J12-Pad1)
- JP3 pad 1: /Vbb_in -> Net-(J5-Pad6)
- JP3 pad 2: /BB_DC -> GND
- JP4 pad 1: GNDD -> Net-(JP4-Pad1)
- JP4 pad 2: /LPWR_LDO -> GND
- L1 pad 1: /ANT -> Net-(L1-Pad1)
- L1 pad 2: /RF_out -> /mcu/DEC4
- L2 pad 1: /DCC -> /mcu/DCC
- L2 pad 2: Net-(L2-Pad2) -> Net-(L1-Pad1)
- L3 pad 1: Net-(L2-Pad2) -> /mcu/ANT
- L3 pad 2: /DEC4 -> /mcu/RF_out
- L4 pad 1: /Vboost_in -> +5V
- L4 pad 2: /Boost_SW -> /dc_boost/Boost_SW
- L5 pad 1: /BB_SWE -> /solar/BB_SWE
- L5 pad 2: GNDD -> +5V
- R1 pad 1: /Vnrf -> Net-(J12-Pad1)
- R1 pad 2: /nRESET -> /P02
- R10 pad 1: /BB_DC -> Net-(R10-Pad1)
- R10 pad 2: /Vbb_in -> +2V8
- R11 pad 1: /BB_FB -> GND
- R11 pad 2: GND -> Net-(R10-Pad1)
- R12 pad 1: GNDD -> Net-(R12-Pad1)
- R12 pad 2: /BB_FB -> Net-(R10-Pad1)
- R2 pad 1: +5V -> /P02
- R2 pad 2: /Boost_FB -> GND
- R3 pad 1: /Boost_FB -> Net-(J13-Pad1)
- R3 pad 2: GND -> /P03
- R4 pad 1: /TP4056_Vcc -> /P03
- R4 pad 2: Net-(JP2-Pad2) -> GND
- R5 pad 1: Net-(JP2-Pad2) -> Net-(J14-Pad1)
- R5 pad 2: GND -> /P04
- R6 pad 1: Net-(R6-Pad1) -> /P16
- R6 pad 2: GND -> Net-(D1-Pad3)
- R7 pad 1: GND -> /P17
- R7 pad 2: /TP4056_Vcc -> Net-(D1-Pad4)
- R8 pad 1: Net-(R8-Pad1) -> /P18
- R8 pad 2: Net-(D1-Pad4) -> Net-(D1-Pad1)
- R9 pad 1: Net-(R9-Pad1) -> /SD_EN
- R9 pad 2: Net-(D1-Pad3) -> GND
- RV1 pad 2: /Boost_FB -> /dc_boost/Boost_FB
- RV1 pad 3: +5V -> +12V
- RV2 pad 1: GNDD -> +5V
- RV2 pad 2: /BB_FB -> /solar/BB_FB
- SC1 pad 1: /Vbb_in -> /solar/SOLAR+
- SC1 pad 2: GNDD -> +5V
- SW1 pad 2: /nRESET -> /RESET
- TP1 pad 1: /nRESET -> +2V8
- TP2 pad 1: Net-(C1-Pad1) -> Net-(C15-Pad1)
- TP3 pad 1: Net-(C2-Pad1) -> Net-(C14-Pad1)
- TP4 pad 1: /Vnrf -> /RESET
- U1 pad 1: /DEC1 -> Net-(J2-Pad2)
- U1 pad 2: Net-(U1-Pad2) -> Net-(J2-Pad1)
- U1 pad 3: Net-(U1-Pad3) -> +12V
- U1 pad 4: Net-(U1-Pad4) -> GND
- U2 pad 2: +3V3 -> +5V
- U2 pad 3: /Vreg -> +12V
- U3 pad 1: /Boost_SW -> GND
- U3 pad 2: GND -> /P02
- U3 pad 3: /Boost_FB -> +5V
- U4 pad 1: Net-(JP2-Pad2) -> /ULN1
- U4 pad 2: Net-(R6-Pad1) -> /ULN2
- U4 pad 3: GND -> /AOP1
- U4 pad 4: /TP4056_Vcc -> /AOP2
- U4 pad 5: /Vbat -> /AOP_EN
- U4 pad 6: Net-(R8-Pad1) -> /P29
- U4 pad 7: Net-(R9-Pad1) -> /P30
- U4 pad 8: /TP4056_Vcc -> GND
- U5 pad 1: /BB_DC -> /AOP1
- U5 pad 2: /BB_SWE -> /capacitive_sensor/MPR0
- U5 pad 3: /BB_TC -> Net-(R12-Pad1)
- U5 pad 4: GNDD -> Net-(JP4-Pad1)
- U5 pad 5: /BB_FB -> Net-(R13-Pad1)
- U5 pad 6: /Vbb_in -> /capacitive_sensor/MPR1
- U5 pad 7: /BB_DC -> /AOP2
- U5 pad 8: /BB_DC -> +2V8
- U6 pad 1: GND -> /MPR_nIRQ
- U6 pad 2: /LPWR_LDO -> /SCL
- U6 pad 3: +2V8 -> /SDA
- U7 pad 1: /Vnrf -> /mcu/DEC1
- U7 pad 2: /SWDIO -> /P00
- U7 pad 3: /nRESET -> /P01
- U7 pad 4: /SWDCLK -> /P02
- U7 pad 5: GND -> /P03
- U7 pad 6: Net-(U7-Pad6) -> /P04
- U8 pad 1: Net-(J1-Pad2) -> +2V8
- U8 pad 2: Net-(J1-Pad1) -> /mcu/SWDIO
- U8 pad 3: /Vreg -> /RESET
- U8 pad 4: GND -> /mcu/SWDCLK
- U9 pad 1: GND -> /dc_boost/Boost_SW
- U9 pad 2: /TEMP_DQ -> GND
- U9 pad 3: +5V -> /dc_boost/Boost_FB
- Y1 pad 1: Net-(C1-Pad1) -> /P00
- Y1 pad 2: Net-(C2-Pad1) -> /P01
Routing:
- net /Vnrf: track 26.8 -> 0.00 mm, vias 3 -> 0
- net +2V8: track 0.00 -> 24.6 mm, vias 0 -> 3
- net Net-(C14-Pad1): track 0.00 -> 16.9 mm
- net Net-(C2-Pad1): track 11.5 -> 0.00 mm
- net Net-(C15-Pad1): track 0.00 -> 11.3 mm
- net Net-(C1-Pad1): track 10.5 -> 0.00 mm
- net /mcu/ANT: track 0.00 -> 7.09 mm
- net /ANT: track 7.09 -> 0.00 mm
- net /P00: track 0.00 -> 5.67 mm
- net /P01: track 0.00 -> 5.46 mm
- net /DEC4: track 4.18 -> 0.00 mm, vias 1 -> 0
- net /mcu/DEC4: track 0.00 -> 3.82 mm, vias 0 -> 1
- net /mcu/DEC2: track 0.00 -> 2.87 mm
- net /DEC2: track 2.87 -> 0.00 mm
- net /mcu/RF_out: track 0.00 -> 2.15 mm
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Other:
- board outline added: 68.6 x 53.4 mm

Commit message: finished placing
Parts:
- removed RV1, RV2: R_POT, Potentiometer_THT:Potentiometer_Runtron_RM-065_Vertical
- removed TH2: NTC, smdpad:smdpad_01x02_1.27_2.54_0.51
- added C28: 10nF, Capacitor_SMD:C_0201_0603Metric, B.Cu at (61.6, 53.7)
- added C29: 0.1uF, Capacitor_SMD:C_0201_0603Metric, B.Cu at (61.6, 55.3)
- added C30: 0.1uF, Capacitor_SMD:C_0201_0603Metric, B.Cu at (63.6, 56.5)
- added C31: C, Capacitor_SMD:C_0201_0603Metric, B.Cu at (28.5, 63.2)
- added C32: CP, Capacitor_SMD:CP_Elec_4x3, F.Cu at (32.6, 30.6)
- added D8: LED, LED_SMD:LED_0603_1608Metric, F.Cu at (33.2, 72.6)
- added J15: Conn_01x08, smdpad:smdpad_01x08_1.27_2.54_0.51, B.Cu at (74.4, 31.5)
- added JP12: TempEN, Jumper:SolderJumper-2_P1.3mm_Bridged_RoundedPad1.0x1.5mm, F.Cu at (32.4, 38.2)
- added JP13: shunt, Jumper:SolderJumper-2_P1.3mm_Open_TrianglePad1.0x1.5mm, B.Cu at (32.5, 45.4)
- added JP14: Vbat, Jumper:SolderJumper-3_P1.3mm_Bridged12_RoundedPad1.0x1.5mm, B.Cu at (32.3, 52.3)
- added JP15: Vmpr, Jumper:SolderJumper-2_P1.3mm_Bridged_RoundedPad1.0x1.5mm, F.Cu at (65.6, 58.9)
- added JP16: Vaop, Jumper:SolderJumper-2_P1.3mm_Bridged_RoundedPad1.0x1.5mm, B.Cu at (66.3, 68.7)
- added JP17: Vsd, Jumper:SolderJumper-2_P1.3mm_Bridged_RoundedPad1.0x1.5mm, B.Cu at (47.8, 67.4)
- added L6: >=26uH, Inductor_SMD:L_Bourns-SRN6028, B.Cu at (28.0, 70.4)
- added Q4: 2N7002, Package_TO_SOT_SMD:SOT-23, F.Cu at (60.2, 41.5)
- added Q5: 2N7002, Package_TO_SOT_SMD:SOT-23, F.Cu at (60.2, 37.5)
- added R43: R, Resistor_SMD:R_0201_0603Metric, B.Cu at (33.0, 61.3)
- added R44: R, Resistor_SMD:R_0201_0603Metric, B.Cu at (33.7, 60.6)
- added R45: R, Resistor_SMD:R_0201_0603Metric, B.Cu at (28.7, 64.5)
- added R46: R, Resistor_SMD:R_0201_0603Metric, B.Cu at (27.9, 64.5)
- added R47: R, Resistor_SMD:R_0201_0603Metric, B.Cu at (31.5, 61.3)
- added R48: R, Resistor_SMD:R_0201_0603Metric, B.Cu at (30.0, 61.3)
- added R49: R, Resistor_SMD:R_0201_0603Metric, B.Cu at (33.0, 59.7)
- added R50: R, Resistor_SMD:R_0201_0603Metric, B.Cu at (34.2, 61.7)
- added R51: R, Resistor_SMD:R_0201_0603Metric, B.Cu at (34.5, 62.9)
- added R52: R, Resistor_SMD:R_0201_0603Metric, B.Cu at (34.4, 64.3)
- added TH1: NTC, smdpad:smdpad_01x02_1.27_1.27_0.51, F.Cu at (32.5, 35.6)
- added TP10: MPR_EN, TestPoint:TestPoint_Pad_D1.0mm, F.Cu at (57.8, 58.7)
- added TP11: SD_EN, TestPoint:TestPoint_Pad_D1.0mm, F.Cu at (47.4, 59.6)
- added TP12: AOP_EN, TestPoint:TestPoint_Pad_D1.0mm, F.Cu at (53.1, 62.5)
- added TP13: Vbat, TestPoint:TestPoint_Pad_D1.0mm, F.Cu at (58.4, 49.4)
- added TP14: AOP1, TestPoint:TestPoint_Pad_D1.0mm, F.Cu at (58.9, 66.2)
- added TP15: AOP2, TestPoint:TestPoint_Pad_D1.0mm, F.Cu at (66.2, 65.5)
- added TP16: Vbridge, TestPoint:TestPoint_Pad_D1.0mm, F.Cu at (52.2, 57.4)
- added TP17: Rx, TestPoint:TestPoint_Pad_D1.0mm, F.Cu at (86.1, 30.5)
- added TP18: Tx, TestPoint:TestPoint_Pad_D1.0mm, F.Cu at (83.4, 30.5)
- added TP21: PRESSURE_CS, TestPoint:TestPoint_Pad_D1.0mm, F.Cu at (43.4, 70.0)
- added TP22: MISO, TestPoint:TestPoint_Pad_D1.0mm, F.Cu at (47.2, 70.1)
- added TP23: ACC_nCS, TestPoint:TestPoint_Pad_D1.0mm, F.Cu at (62.7, 58.7)
- added TP24: MOSI, TestPoint:TestPoint_Pad_D1.0mm, F.Cu at (43.7, 72.4)
- added TP25: MOSI, TestPoint:TestPoint_Pad_D1.0mm, F.Cu at (46.0, 72.3)
- added TP26: TEMP_DQ, TestPoint:TestPoint_Pad_D1.0mm, F.Cu at (54.5, 58.4)
- added TP27: Vsolar, TestPoint:TestPoint_Pad_D1.0mm, F.Cu at (34.9, 25.5)
- added TP28: VinDC, TestPoint:TestPoint_Pad_D1.0mm, F.Cu at (39.2, 30.5)
- added TP29: BoostEN, TestPoint:TestPoint_Pad_D1.0mm, F.Cu at (52.8, 34.9)
- added TP30: BoostVin, TestPoint:TestPoint_Pad_D1.0mm, F.Cu at (55.2, 38.2)
- added TP31: SW, TestPoint:TestPoint_Pad_D1.0mm, F.Cu at (47.2, 38.9)
- added TP32: Vout, TestPoint:TestPoint_Pad_D1.0mm, F.Cu at (48.3, 31.1)
- added TP33: BoostFB, TestPoint:TestPoint_Pad_D1.0mm, F.Cu at (52.5, 32.6)
- added TP5: SCL, TestPoint:TestPoint_Pad_D1.0mm, F.Cu at (67.9, 55.8)
- added TP6: GNDD, TestPoint:TestPoint_Pad_D1.0mm, B.Cu at (25.7, 48.3)
- added TP7: BB_FB, TestPoint:TestPoint_Pad_D1.0mm, B.Cu at (34.0, 48.5)
- added TP8: GND, TestPoint:TestPoint_Pad_D1.0mm, B.Cu at (35.8, 49.8)
- added TP9: SDA, TestPoint:TestPoint_Pad_D1.0mm, F.Cu at (70.1, 55.9)
- added U17: MPU-9250, Sensor_Motion:InvenSense_QFN-24_3x3mm_P0.4mm, B.Cu at (64.2, 53.9)
- added U18: BQ25504, Package_DFN_QFN:QFN-16-1EP_3x3mm_P0.5mm_EP1.7x1.7mm, B.Cu at (31.5, 64.0)
- BT1: footprint Connector_PinHeader_2.54mm:PinHeader_1x02_P2.54mm_Vertical -> smdpad:smdpad_01x02_2.54_2.54_0.51
- C17, C18, C24, C25, C26, C27, D2, J3, JP10, JP11, JP2, JP9, L4, Q2, U15, U16, U5, U9: moved to B.Cu
- C21: footprint Capacitor_THT:CP_Radial_D10.0mm_P5.00mm -> Capacitor_SMD:CP_Elec_4x3
- C22: footprint Capacitor_SMD:C_0201_0603Metric -> Capacitor_SMD:CP_Elec_4x3
- Csd1: footprint Capacitor_SMD:C_Elec_6.3x5.4 -> Capacitor_SMD:CP_Elec_4x3
- D5, D6, D7: footprint LED_SMD:LED_1210_3225Metric -> LED_SMD:LED_0603_1608Metric
- H1, H2, H3, H4: footprint MountingHole:MountingHole_2.2mm_M2_DIN965_Pad -> MountingHole:MountingHole_2.2mm_M2_DIN965_Pad_TopBottom
- J1: footprint Connector_PinHeader_2.54mm:PinHeader_1x04_P2.54mm_Vertical -> smdpad:smdpad_01x04_1.27_2.54_0.51; moved to B.Cu
- J2: footprint smdpad:smdpad_01x02_2.54_3.81_2.54 -> smdpad:smdpad_01x02_1.27_2.54_0.51; moved to B.Cu
- JP1: moved to F.Cu
- JP4: value AOP_EN -> Vacc; footprint Jumper:SolderJumper-2_P1.3mm_Open_TrianglePad1.0x1.5mm -> Jumper:SolderJumper-2_P1.3mm_Bridged_RoundedPad1.0x1.5mm
- JP5: value AOP_EN -> Vbat; footprint Jumper:SolderJumper-2_P1.3mm_Open_TrianglePad1.0x1.5mm -> Jumper:SolderJumper-3_P1.3mm_Bridged12_RoundedPad1.0x1.5mm; moved to B.Cu
- JP6: value TempEN -> Vsd
- JP7: value shunt -> Boost_in; footprint Jumper:SolderJumper-2_P1.3mm_Open_TrianglePad1.0x1.5mm -> Jumper:SolderJumper-3_P1.3mm_Bridged12_RoundedPad1.0x1.5mm; moved to B.Cu
- JP8: value Vbat -> Boost_out
- L5: footprint Inductor_SMD:L_Coilcraft_XAL60xx_6.36x6.56mm -> Inductor_SMD:L_Bourns-SRN6028
- R1, R2, R20, R21, R22, R23, R24, R25, R26, R29, R3, R30, R31, R32, R33, R34, R35, R36, R37, R39, R4, R40, R41, R42, R5, R6, R7, R8, R9: footprint Resistor_SMD:R_0805_2012Metric -> Resistor_SMD:R_0201_0603Metric
- R10, R11, R12, R13, R14, R15, R16, R17, R18, R19, R27, R28, R38: footprint Resistor_SMD:R_0805_2012Metric -> Resistor_SMD:R_0201_0603Metric; moved to B.Cu
- U1: value WX-DC12003 -> ULN2003; footprint aliexpress:WX-DC12003_vertical -> Package_SO:STC_SOP-16_3.9x9.9mm_P1.27mm; moved to B.Cu
- moved J2 258.9 mm to (25.7, 26.4), turned to 180 degrees
- moved J3 249.8 mm to (27.7, 37.8), turned to 90 degrees
- moved JP5 246.3 mm to (26.0, 63.9), turned to 90 degrees
- moved J13 239.6 mm to (51.2, 49.9), turned to 90 degrees
- moved J14 236.3 mm to (51.2, 44.3), turned to 90 degrees
- moved R7 233.1 mm to (65.9, 49.1), turned to 270 degrees
- moved JP10 232.8 mm to (58.9, 54.0), turned to 90 degrees
- moved J12 232.2 mm to (51.2, 55.5), turned to 90 degrees
- moved U4 232.0 mm to (68.3, 38.4), turned to 90 degrees
- moved D1 223.8 mm to (63.6, 47.6), turned to 270 degrees
- moved J6 223.1 mm to (62.0, 31.5)
- moved U16 220.2 mm to (33.0, 37.1)
- moved C27 218.3 mm to (29.8, 35.3), turned to 90 degrees
- moved C26 215.0 mm to (31.4, 34.0), turned to 180 degrees
- moved R38 213.9 mm to (32.9, 33.5), turned to 270 degrees
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Connections:
- net /battery_charger/TP4056_Vcc renamed /power_management/sheet618CA8D9/TP4056_Vcc
- net /dc_boost/Boost_FB renamed /power_management/sheet618CA8D8/Boost_FB
- net /dc_boost/Boost_SW renamed /power_management/sheet618CA8D8/Boost_SW
- net /solar/BB_FB renamed /power_management/sheet618CA8DA/BB_FB
- net /solar/BB_SWE renamed /power_management/sheet618CA8DA/BB_SWE
- net /solar/BB_TC renamed /power_management/sheet618CA8DA/BB_TC
- BT1 pad 1: /Vbat -> /power_management/Vbat
- C17 pad 1: +5V -> /power_management/sheet618CA8D8/Vin
- C18 pad 1: +12V -> /power_management/sheet618CA8D8/Vout
- C19 pad 1: /Vbat -> /power_management/Vbat
- C2 pad 1: +2V8 -> /capacitive_sensor/Vmpr
- C22 pad 1: +2V8 -> +3V3
- C23 pad 1: +2V8 -> /Vacc
- C24 pad 1: +2V8 -> /pressure_sensor/Vin
- C25 pad 2: +2V8 -> /pressure_sensor/Vin
- C5 pad 1: +2V8 -> +3V3
- C6 pad 1: +2V8 -> +3V3
- C7 pad 1: +2V8 -> +3V3
- C8 pad 1: +2V8 -> +3V3
- Csd1 pad 1: +2V8 -> /interfaces/Vsd
- D1 pad 2: +2V8 -> +3V3
- D2 pad 1: +12V -> /power_management/sheet618CA8D8/Vout
- J10 pad 3: +2V8 -> +3V3
- J2 pad 1: Net-(J2-Pad1) -> /power_management/VinDC
- J2 pad 2: Net-(J2-Pad2) -> GND
- J3 pad 10: +2V8 -> +3V3
- J3 pad 2: +2V8 -> +12V
- J3 pad 4: +12V -> /VAC
- J3 pad 8: +2V8 -> +3V3
- J5 pad 4: +2V8 -> /interfaces/Vsd
- J8 pad 2: +2V8 -> +3V3
- J8 pad 4: +2V8 -> +3V3
- J8 pad 8: +2V8 -> +3V3
- JP10 pad 1: +2V8 -> +3V3
- JP4 pad 1: Net-(JP4-Pad1) -> +3V3
- JP4 pad 2: GND -> /Vacc
- JP5 pad 1: /capacitive_sensor/MPR_Vss -> +5V
- JP5 pad 2: GND -> /power_management/sheet618CA8DA/SOLAR-
- JP6 pad 1: GND -> +3V3
- JP6 pad 2: Net-(JP6-Pad2) -> /interfaces/Vsd
- JP7 pad 1: /solar/SOLAR+ -> +5V
- JP7 pad 2: /solar/BB_DC -> /power_management/sheet618CA8D8/Vin
- JP8 pad 1: /Vbat -> /power_management/VinDC
- JP8 pad 2: Net-(JP8-Pad2) -> /power_management/sheet618CA8D8/Vout
- L4 pad 1: +5V -> /power_management/sheet618CA8D8/Vin
- Q2 pad 3: Net-(JP4-Pad1) -> Net-(Q2-Pad3)
- R10 pad 2: +2V8 -> /capacitive_sensor/Vaop
- R18 pad 1: +2V8 -> /capacitive_sensor/Vaop
- R24 pad 1: +2V8 -> /capacitive_sensor/Vmpr
- R26 pad 1: +2V8 -> +3V3
- R27 pad 1: +12V -> /power_management/sheet618CA8D8/Vout
- R29 pad 2: Net-(JP6-Pad2) -> Net-(JP12-Pad2)
- R30 pad 1: Net-(JP6-Pad2) -> Net-(JP12-Pad2)
- R35 pad 1: /solar/BB_DC -> /power_management/sheet618CA8DA/BB_DC
- R35 pad 2: /solar/SOLAR+ -> /power_management/sheet618CA8DA/SOLAR+
- R40 pad 1: +2V8 -> +3V3
- R41 pad 1: +2V8 -> +3V3
- R42 pad 1: +2V8 -> +3V3
- SC1 pad 1: /solar/SOLAR+ -> /power_management/sheet618CA8DA/SOLAR+
- SC1 pad 2: +5V -> /power_management/sheet618CA8DA/SOLAR-
- TP1 pad 1: +2V8 -> +3V3
- U1 pad 1: Net-(J2-Pad2) -> /SCL
- U1 pad 2: Net-(J2-Pad1) -> /SDA
- U1 pad 3: +12V -> /Rx
- U1 pad 4: GND -> /P03
- U10 pad 1: Net-(JP6-Pad2) -> Net-(JP12-Pad2)
- U10 pad 5: /Vbat -> /power_management/Vbat
- U11 pad 1: /solar/BB_DC -> /power_management/sheet618CA8DA/BB_DC
- U11 pad 6: /solar/SOLAR+ -> /power_management/sheet618CA8DA/SOLAR+
- U11 pad 7: /solar/BB_DC -> /power_management/sheet618CA8DA/BB_DC
- U11 pad 8: /solar/BB_DC -> /power_management/sheet618CA8DA/BB_DC
- U12 pad 2: Net-(JP8-Pad2) -> Net-(JP14-Pad2)
- U12 pad 3: +2V8 -> +3V3
- U13 pad 2: +2V8 -> +3V3
- U13 pad 3: Net-(JP8-Pad2) -> Net-(JP14-Pad2)
- U14 pad 1: +2V8 -> /Vacc
- U14 pad 6: +2V8 -> /Vacc
- U15 pad 6: +2V8 -> /pressure_sensor/Vin
- U15 pad 8: +2V8 -> /pressure_sensor/Vin
- U2 pad 3: +12V -> /power_management/VinDC
- U5 pad 4: Net-(JP4-Pad1) -> Net-(Q2-Pad3)
- U5 pad 8: +2V8 -> /capacitive_sensor/Vaop
- U6 pad 20: +2V8 -> /capacitive_sensor/Vmpr
- U7 pad 13: +2V8 -> +3V3
- U7 pad 36: +2V8 -> +3V3
- U7 pad 48: +2V8 -> +3V3
- U8 pad 1: +2V8 -> +3V3
- U9 pad 4: /BOOST_EN -> /power_management/BOOST_EN
- U9 pad 5: +5V -> /power_management/sheet618CA8D8/Vin
Routing:
- net +3V3: track 0.00 -> 24.6 mm, vias 0 -> 3
- net +2V8: track 24.6 -> 0.00 mm, vias 3 -> 0
- added copper zone on B.Cu, net GND
- added copper zone on F.Cu, net GND
Other:
- outline, holes or cut-outs redrawn
- net class Default: clearance 0.13 -> 0.127; trace_width 0.1524 -> 0.13; via_dia 0.4 -> 0.6; via_drill 0.2 -> 0.3
- net class PWR: trace_width 0.2 -> 0.13; via_dia 0.4 -> 0.6; via_drill 0.2 -> 0.3
- rule trace_clearance: 0.13 -> 0.127
- rule trace_min: 0.127 -> 0.13
- rule via_min_drill: 0.2 -> 0.3
- rule via_min_size: 0.4 -> 0.6

Commit message: antenna connexion
Routing:
- net GND: track 10.4 -> 14.9 mm
Changed lines of the file:
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@@
     (thickness 1.6)
     (drawings 8)
-    (tracks 91)
+    (tracks 94)
     (zones 0)
     (modules 196)
@@
   )
   (setup
-    (last_trace_width 0.13)
+    (last_trace_width 0.6)
     (user_trace_width 0.2)
+    (user_trace_width 0.6)
+    (user_trace_width 0.8)
+    (user_trace_width 1)
     (trace_clearance 0.127)
     (zone_clearance 0.508)
@@
   (gr_line (start 22.606 24.384) (end 88.646 24.384) (layer Edge.Cuts) (width 0.05))
   (gr_line (start 22.558 77.738) (end 22.606 24.384) (layer Edge.Cuts) (width 0.05))
+  (segment (start 90.2462 50.3936) (end 90.2462 51.6636) (width 0.6) (layer F.Cu) (net 1))
   (segment (start 76.527 52.378) (end 76.327 52.578) (width 0.2) (layer F.Cu) (net 1))
   (segment (start 79.277 52.378) (end 76.527 52.378) (width 0.2) (layer F.Cu) (net 1))
@@
   (segment (start 74.6048 47.0916) (end 74.9808 47.4676) (width 0.2) (layer F.Cu) (net 1))
   (segment (start 73.7108 47.0916) (end 74.6048 47.0916) (width 0.2) (layer F.Cu) (net 1))
+  (segment (start 89.557 60.462) (end 89.557 62.4552) (width 1) (layer F.Cu) (net 1))
+  (segment (start 87.457 58.112) (end 86.1854 58.112) (width 0.6) (layer F.Cu) (net 1))
   (segment (start 82.41001 52.77119) (end 82.41001 52.7812) (width 0.8) (layer F.Cu) (net 11))
   (segment (start 82.4254 52.7558) (end 82.41001 52.77119) (width 0.8) (layer F.Cu) (net 11))
@@
     (connect_pads (clearance 0.508))
     (min_thickness 0.254)
-    (keepout (tracks not_allowed) (vias not_allowed) (copperpour not_allowed))
+    (keepout (tracks allowed) (vias not_allowed) (copperpour not_allowed))
     (fill (arc_segments 32) (thermal_gap 0.508) (thermal_bridge_width 0.508))
     (polygon

Commit message: wip routage
Parts:
- moved R6 4.55 mm to (61.6, 44.6), turned to 180 degrees
- moved R7 4.28 mm to (61.6, 49.2), turned to 180 degrees
- moved TP12 4.12 mm to (52.0, 66.5)
- moved C4 3.69 mm to (67.4, 50.5), turned to 90 degrees
- moved R8 3.67 mm to (65.1, 49.2), turned to 180 degrees
- moved C1 3.58 mm to (57.8, 63.3), turned to 90 degrees
- moved C2 3.06 mm to (62.6, 65.1)
- moved R23 3.06 mm to (57.2, 65.9)
- moved TP15 3.06 mm to (63.5, 67.0)
- moved R17 3.06 mm to (64.8, 64.4)
- moved R25 3.06 mm to (53.2, 64.2)
- moved U5 3.06 mm to (60.4, 65.3)
- moved Q3 3.06 mm to (55.5, 63.6)
- moved R10 3.06 mm to (61.2, 61.1)
- moved R13 3.06 mm to (61.2, 61.8)
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Routing:
- net +3V3: track 24.6 -> 219.4 mm, vias 3 -> 12
- net +5V: track 0.00 -> 180.5 mm, vias 0 -> 7
- net /SCL: track 0.00 -> 158.3 mm, vias 0 -> 7
- net /SDA: track 0.00 -> 150.8 mm, vias 0 -> 11
- net /PRESSURE_CS: track 0.00 -> 126.9 mm, vias 0 -> 3
- net /Rx: track 0.00 -> 125.1 mm, vias 0 -> 2
- net /AOP1: track 0.00 -> 107.4 mm, vias 0 -> 9
- net /SD_EN: track 0.00 -> 106.7 mm, vias 0 -> 4
- net /AOP_EN: track 0.00 -> 101.2 mm, vias 0 -> 7
- net /P03: track 0.00 -> 100.8 mm, vias 0 -> 3
- net /P04: track 0.00 -> 100.2 mm, vias 0 -> 9
- net /ULN2: track 0.00 -> 98.2 mm, vias 0 -> 5
- net /MISO: track 0.00 -> 95.9 mm, vias 0 -> 8
- net /Tx: track 0.00 -> 95.5 mm, vias 0 -> 2
- net /MPR_EN: track 0.00 -> 91.2 mm, vias 0 -> 2
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Other:
- net class Default: clearance 0.127 -> 0.13
- net class PWR: trace_width 0.13 -> 0.2
- rule trace_clearance: 0.127 -> 0.13

Commit message: finished routing
Parts:
- J3: footprint smdpad:smdpad_02x05_1.27_2.54_0.51 -> smdpad:smdpad_02x04_1.27_2.54_0.51
- moved TP5 12.9 mm to (71.6, 68.2)
- moved J3 6.70 mm to (24.7, 31.9), turned to 270 degrees
- moved TP23 3.75 mm to (65.4, 61.3)
- moved C27 3.53 mm to (31.0, 32.1)
- moved TP12 1.71 mm to (50.8, 67.7)
- moved C23 1.40 mm to (60.2, 53.0), turned to 180 degrees
- moved TP33 1.35 mm to (53.6, 31.5)
- moved TP9 1.11 mm to (70.4, 57.0)
- moved C6 0.78 mm to (72.6, 47.1)
- moved C28 0.66 mm to (60.9, 53.6)
- moved C8 0.65 mm to (73.1, 56.7), turned to 0 degrees
- moved C3 0.49 mm to (70.8, 48.3), turned to 90 degrees
- moved C9 0.33 mm to (75.0, 47.5)
- moved C11 0.24 mm to (82.3, 51.5)
Connections:
- J1 pad 2: /US_ECHO -> /ACC_INT1
- J1 pad 3: /US_TRIG -> /ACC_INT2
- J2 pad 1: /power_management/VinDC -> /VinDC
- J3 pad 1: +5V -> +3V3
- J3 pad 2: +12V -> +3V3
- J3 pad 3: /Vbb_in -> /Vbat
- J3 pad 4: /VAC -> +5V
- J3 pad 5: +5V -> GND
- J3 pad 6: GND -> Net-(J3-Pad6)
- J3 pad 7: /Vbat -> /VinDC
- J3 pad 8: +3V3 -> +5V
- JP8 pad 1: /power_management/VinDC -> /VinDC
- TP28 pad 1: /power_management/VinDC -> /VinDC
- U16 pad 5: Net-(U16-Pad5) -> +3V3
- U2 pad 3: /power_management/VinDC -> /VinDC
- U7 pad 22: /US_ECHO -> /ACC_INT1
- U7 pad 23: /US_TRIG -> /ACC_INT2
Routing:
- net /VinDC: track 0.00 -> 48.7 mm, vias 0 -> 3
- net /ACC_INT1: track 4.80 -> 50.3 mm, vias 1 -> 7
- net /ACC_INT2: track 0.00 -> 44.5 mm, vias 0 -> 5
- net GND: track 36.3 -> 69.0 mm, vias 66 -> 109
- net /power_management/VinDC: track 27.9 -> 0.00 mm, vias 1 -> 0
- net /capacitive_sensor/MPR1: track 41.1 -> 15.6 mm
- net /US_TRIG: track 24.7 -> 0.00 mm, vias 3 -> 0
- net /US_ECHO: track 21.5 -> 0.00 mm, vias 3 -> 0
- net +3V3: track 219.4 -> 235.9 mm, vias 12 -> 15
- net /SCL: track 158.3 -> 169.1 mm
- net +5V: track 180.5 -> 190.4 mm, vias 7 -> 8
- net /P16: track 59.4 -> 65.6 mm, vias 2 -> 4
- net /power_management/sheet618CA8DA/OK_HIST: track 5.11 -> 10.1 mm
- net /SD_CS: track 76.3 -> 81.0 mm
- net /power_management/Vbat: track 71.6 -> 75.8 mm
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
Commit message: WIP silkscreen
Other:
- board text added: "+"
- board text added: "-"
- board text added: "Flash"
- board text added: "Micro SDCard"
- board text added: "USB"
